File: board/RPi_Hat.kicad_pcb (KiCad board)
At the start: 2 copper layers, 65 x 56 mm, 5 parts, among them J1 PiHat

Commit message: finished schematic
Parts:
- added A1: Sparkfun-CCS811, HWP:Sparkfun-CCS881, F.Cu at (8.98, 1.36)
- added A2: BME280, HWP:BME280, F.Cu at (13.9, 40.5)
- added C1: 100n, HWP:C_0805, F.Cu at (7.62, 37.1)
- added D1: red, HWP:LED_0805, F.Cu at (-93.5, 52.9)
- added D2: red, HWP:LED_0805, F.Cu at (-93.5, 49.8)
- added D3: red, HWP:LED_0805, F.Cu at (-82.0, 41.3)
- added D4: red, HWP:LED_0805, F.Cu at (-103.0, 52.9)
- added D5: red, HWP:LED_0805, F.Cu at (-98.3, 52.9)
- added D6: red, HWP:LED_0805, F.Cu at (-60.5, 29.3)
- added D7: red, HWP:LED_0805, F.Cu at (-98.3, 49.8)
- added D8: red, HWP:LED_0805, F.Cu at (61.0, 12.7)
- added DS1: OLED, HWP:OLED, F.Cu at (43.4, 29.0)
- added R1: 10k, HWP:R_0805, F.Cu at (-28.9, 15.1)
- added R10: 10k, HWP:R_0805, F.Cu at (-44.9, 29.2)
- added R11: 150, HWP:R_0805, F.Cu at (-74.5, 52.8)
- added R12: 150, HWP:R_0805, F.Cu at (-79.2, 52.8)
- added R13: 150, HWP:R_0805, F.Cu at (-88.7, 52.7)
- added R14: 150, HWP:R_0805, F.Cu at (-84.0, 53.1)
- added R15: 150, HWP:R_0805, F.Cu at (-28.9, 12.1)
- added R16: 150, HWP:R_0805, F.Cu at (-55.5, 37.8)
- added R17: 150, HWP:R_0805, F.Cu at (-84.0, 50.2)
- added R18: 150, HWP:R_0805, F.Cu at (-44.9, 32.2)
- added R2: 10k, HWP:R_0805, F.Cu at (-39.5, 23.6)
- added R3: 10k, HWP:R_0805, F.Cu at (-39.5, 20.7)
- added R4: 10k, HWP:R_0805, F.Cu at (-82.0, 47.2)
- added R5: 10k, HWP:R_0805, F.Cu at (-39.5, 26.6)
- added R6: 10k, HWP:R_0805, F.Cu at (-69.7, 52.8)
- added R7: 10k, HWP:R_0805, F.Cu at (-82.0, 44.3)
- added R8: 10k, HWP:R_0805, F.Cu at (-55.5, 40.7)
- added R9: 10k, HWP:R_0805, F.Cu at (-88.7, 49.8)
- added SW1: Pushbutton, HWP:PushButton, F.Cu at (17.8, 33.0)
- added SW2: Pushbutton, HWP:PushButton, F.Cu at (29.8, 33.3)
- added SW3: Pushbutton, HWP:PushButton, F.Cu at (39.9, 33.3)
- added SW4: Pushbutton, HWP:PushButton, F.Cu at (53.3, 33.3)
- added SW5: Pushbutton, HWP:PushButton, F.Cu at (12.7, 46.0)
- added SW6: Pushbutton, HWP:PushButton, F.Cu at (24.7, 46.0)
- added SW7: Pushbutton, HWP:PushButton, F.Cu at (37.4, 46.0)
- added SW8: Pushbutton, HWP:PushButton, F.Cu at (50.1, 46.0)
Connections:
- J1 pad 1: Net-(J1-Pad1) -> +3V3
- J1 pad 10: Net-(J1-Pad10) -> unconnected-(J1-Pad10)
- J1 pad 11: Net-(J1-Pad11) -> unconnected-(J1-Pad11)
- J1 pad 12: Net-(J1-Pad12) -> unconnected-(J1-Pad12)
- J1 pad 13: Net-(J1-Pad13) -> unconnected-(J1-Pad13)
- J1 pad 14: Net-(J1-Pad14) -> GND
- J1 pad 15: Net-(J1-Pad15) -> unconnected-(J1-Pad15)
- J1 pad 16: Net-(J1-Pad16) -> unconnected-(J1-Pad16)
- J1 pad 17: Net-(J1-Pad17) -> +3V3
- J1 pad 18: Net-(J1-Pad18) -> unconnected-(J1-Pad18)
- J1 pad 19: Net-(J1-Pad19) -> unconnected-(J1-Pad19)
- J1 pad 2: Net-(J1-Pad2) -> +5V
- J1 pad 20: Net-(J1-Pad20) -> GND
- J1 pad 21: Net-(J1-Pad21) -> Diode 1
- J1 pad 22: Net-(J1-Pad22) -> Button 1
- J1 pad 23: Net-(J1-Pad23) -> Diode 2
- J1 pad 24: Net-(J1-Pad24) -> Button 2
- J1 pad 25: Net-(J1-Pad25) -> GND
- J1 pad 26: Net-(J1-Pad26) -> Button 3
- J1 pad 27: Net-(J1-Pad27) -> Diode 3
- J1 pad 28: Net-(J1-Pad28) -> Button 4
- J1 pad 29: Net-(J1-Pad29) -> Diode 4
- J1 pad 3: Net-(J1-Pad3) -> SDA
- J1 pad 30: Net-(J1-Pad30) -> GND
- J1 pad 31: Net-(J1-Pad31) -> Diode 5
- J1 pad 32: Net-(J1-Pad32) -> Button 5
- J1 pad 33: Net-(J1-Pad33) -> Diode 6
- J1 pad 34: Net-(J1-Pad34) -> GND
- J1 pad 35: Net-(J1-Pad35) -> Diode 7
- J1 pad 36: Net-(J1-Pad36) -> Button 6
- J1 pad 37: Net-(J1-Pad37) -> Diode 8
- J1 pad 38: Net-(J1-Pad38) -> Button 7
- J1 pad 39: Net-(J1-Pad39) -> GND
- J1 pad 4: Net-(J1-Pad4) -> +5V
- J1 pad 40: Net-(J1-Pad40) -> Button 8
- J1 pad 5: Net-(J1-Pad5) -> SCL
- J1 pad 6: Net-(J1-Pad6) -> GND
- J1 pad 7: Net-(J1-Pad7) -> unconnected-(J1-Pad7)
- J1 pad 8: Net-(J1-Pad8) -> unconnected-(J1-Pad8)
- J1 pad 9: Net-(J1-Pad9) -> GND
Routing:
- net +3V3: track 0.00 -> 10.6 mm
- net GND: track 0.00 -> 10.2 mm
- net +5V: track 0.00 -> 2.54 mm
Other:
- net class Default removed

Commit message: changes
Parts:
- moved D2 209.1 mm to (115.6, 52.1), turned to 90 degrees
- moved D4 192.8 mm to (88.9, 34.3), turned to 90 degrees
- moved D5 188.8 mm to (88.9, 27.9), turned to 90 degrees
- moved D3 176.4 mm to (94.0, 53.6), turned to 90 degrees
- moved D7 176.1 mm to (74.9, 17.8), turned to 90 degrees
- moved D6 147.1 mm to (86.4, 21.6), turned to 90 degrees
- moved R9 126.5 mm to (33.0, 15.2), turned to 90 degrees
- moved R10 52.7 mm to (5.08, 12.7), turned to -90 degrees
- moved D8 28.1 mm to (88.9, 15.2)
- moved R15 23.9 mm to (-6.11, 5.08)
- moved A2 22.1 mm to (25.3, 21.7), turned to -90 degrees
- moved DS1 21.4 mm to (26.8, 15.4), turned to 90 degrees
- moved C1 15.6 mm to (20.3, 27.9)
- moved SW1 12.0 mm to (10.9, 42.9), turned to 180 degrees
- moved SW2 11.4 mm to (23.6, 42.9), turned to 180 degrees
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Routing:
- net SDA: track 0.00 -> 58.7 mm
- net SCL: track 0.00 -> 45.6 mm
- net +3V3: track 10.6 -> 52.5 mm, vias 0 -> 2
- net GND: track 10.2 -> 0.27 mm
- removed copper zone on B.Cu, net GND

Commit message: pcb_completly_wired
Parts:
- moved R17 139.7 mm to (55.2, 37.6), turned to 180 degrees
- moved R7 132.8 mm to (49.6, 26.4), turned to -90 degrees
- moved R13 117.3 mm to (27.5, 37.2), turned to 180 degrees
- moved R6 115.2 mm to (45.5, 53.7), turned to 90 degrees
- moved R4 113.2 mm to (31.0, 53.5), turned to 90 degrees
- moved R14 112.1 mm to (27.8, 44.0), turned to 180 degrees
- moved R8 109.4 mm to (53.0, 54.5)
- moved D2 107.2 mm to (8.75, 43.5), turned to 0 degrees
- moved D1 103.4 mm to (8.75, 37.6)
- moved R18 100.9 mm to (55.2, 43.8), turned to 180 degrees
- moved R16 97.4 mm to (41.8, 43.8), turned to 180 degrees
- moved R12 94.2 mm to (14.5, 43.5), turned to 180 degrees
- moved R11 89.4 mm to (13.6, 37.5), turned to 180 degrees
- moved R5 74.7 mm to (35.2, 26.4), turned to -90 degrees
- moved D3 73.8 mm to (22.0, 37.2), turned to 0 degrees
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Connections:
- J1 pad 22: Button 1 -> Diode 3
- J1 pad 24: Button 2 -> Diode 4
- J1 pad 26: Button 3 -> Diode 5
- J1 pad 27: Diode 3 -> Diode 6
- J1 pad 28: Button 4 -> Diode 7
- J1 pad 29: Diode 4 -> Diode 8
- J1 pad 31: Diode 5 -> Button 3
- J1 pad 33: Diode 6 -> Button 7
- J1 pad 35: Diode 7 -> Button 4
- J1 pad 36: Button 6 -> Button 1
- J1 pad 37: Diode 8 -> Button 6
- J1 pad 38: Button 7 -> Button 2
Routing:
- net +3V3: track 52.5 -> 197.8 mm, vias 2 -> 1
- net Button 1: track 0.00 -> 101.8 mm
- net Button 2: track 0.00 -> 100.4 mm
- net Button 4: track 0.00 -> 85.3 mm
- net Button 3: track 0.00 -> 81.8 mm
- net Button 6: track 0.00 -> 69.8 mm
- net Button 5: track 0.00 -> 68.3 mm
- net Button 8: track 0.00 -> 63.8 mm
- net Diode 2: track 0.00 -> 53.4 mm
- net Diode 1: track 0.00 -> 52.6 mm
- net Diode 8: track 0.00 -> 50.1 mm
- net Diode 7: track 0.00 -> 48.7 mm
- net Diode 4: track 0.00 -> 45.7 mm
- net Diode 5: track 0.00 -> 43.0 mm
- net Diode 6: track 0.00 -> 42.7 mm
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- added copper zone on B.Cu, net GND

Commit message: transistors
Parts:
- removed C1: 100n, HWP:C_0805
- moved SW4 37.1 mm to (56.5, 33.9), turned to 180 degrees
- moved SW5 35.1 mm to (9.35, 47.5), turned to 0 degrees
- moved R4 34.8 mm to (50.0, 24.4), turned to -90 degrees
- moved R5 32.2 mm to (18.9, 54.1), turned to 90 degrees
- moved R14 28.5 mm to (55.5, 37.1)
- moved D4 28.3 mm to (50.5, 37.1)
- moved R2 28.1 mm to (22.4, 25.6), turned to -90 degrees
- moved R7 28.0 mm to (46.1, 54.1), turned to 90 degrees
- moved R15 27.5 mm to (14.8, 44.5)
- moved D5 27.1 mm to (9.85, 44.5)
- moved SW2 23.9 mm to (29.0, 34.0), turned to 180 degrees
- moved SW7 23.5 mm to (36.0, 47.5), turned to 0 degrees
- moved R3 17.9 mm to (39.5, 25.2)
- moved D2 15.6 mm to (23.0, 37.2)
- moved R17 15.3 mm to (41.5, 44.5)
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Connections:
- J1 pad 11: unconnected-(J1-Pad11) -> Diode 2
- J1 pad 13: unconnected-(J1-Pad13) -> Diode 1
- J1 pad 15: unconnected-(J1-Pad15) -> Diode 5
- J1 pad 19: unconnected-(J1-Pad19) -> Diode 6
- J1 pad 21: Diode 1 -> unconnected-(J1-Pad21)
- J1 pad 22: Diode 3 -> unconnected-(J1-Pad22)
- J1 pad 23: Diode 2 -> Diode 4
- J1 pad 24: Diode 4 -> Diode 3
- J1 pad 26: Diode 5 -> unconnected-(J1-Pad26)
- J1 pad 27: Diode 6 -> Diode 7
- J1 pad 28: Diode 7 -> Diode 8
- J1 pad 29: Diode 8 -> Button 4
- J1 pad 31: Button 3 -> Button 2
- J1 pad 32: Button 5 -> Button 3
- J1 pad 33: Button 7 -> Button 1
- J1 pad 35: Button 4 -> Button 6
- J1 pad 36: Button 1 -> Button 5
- J1 pad 37: Button 6 -> Button 7
- J1 pad 38: Button 2 -> Button 8
- J1 pad 40: Button 8 -> unconnected-(J1-Pad40)
Routing:
- net Diode 3: track 36.9 -> 81.6 mm
- net Button 5: track 68.3 -> 109.9 mm
- net Button 7: track 37.3 -> 78.5 mm
- net Button 4: track 85.3 -> 47.4 mm
- net Diode 2: track 53.4 -> 25.6 mm
- net Diode 7: track 48.7 -> 75.0 mm
- net Button 6: track 69.8 -> 92.9 mm
- net Diode 8: track 50.1 -> 64.1 mm
- net Button 1: track 101.8 -> 114.4 mm
- net Diode 6: track 42.7 -> 31.3 mm
- net Diode 4: track 45.7 -> 57.1 mm
- net Button 3: track 81.8 -> 91.0 mm
- net GND: track 8.56 -> 0.00 mm, vias 0 -> 1
- net Diode 1: track 52.6 -> 44.1 mm
- net SCL: track 49.8 -> 55.6 mm
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
Commit message: finalisation
Routing:
- net Diode 5: track 42.0 -> 57.8 mm
- net Diode 1: track 44.1 -> 59.8 mm
- net Diode 6: track 31.3 -> 46.3 mm
- net Diode 2: track 25.6 -> 40.2 mm
Changed lines of the file:
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@@
   (segment (start 41.4 5.24) (end 43.71 7.55) (width 0.25) (layer "F.Cu") (net 24))
   (segment (start 34.2 41.8) (end 31.5 44.5) (width 0.25) (layer "F.Cu") (net 25))
+  (segment (start 29.23 7.25) (end 28.5 7.98) (width 0.25) (layer "F.Cu") (net 25))
   (segment (start 28.5 22.75) (end 34.2 28.45) (width 0.25) (layer "F.Cu") (net 25))
   (segment (start 34.2 28.45) (end 34.2 41.8) (width 0.25) (layer "F.Cu") (net 25))
   (segment (start 31.5 44.5) (end 29.025 44.5) (width 0.25) (layer "F.Cu") (net 25))
-  (segment (start 29.23 7.25) (end 28.5 7.25) (width 0.25) (layer "F.Cu") (net 25))
   (segment (start 31.24 5.24) (end 29.23 7.25) (width 0.25) (layer "F.Cu") (net 25))
+  (segment (start 28.5 7.98) (end 28.5 22.7) (width 0.25) (layer "F.Cu") (net 25))
   (segment (start 17.725 52) (end 18.85 53.125) (width 0.25) (layer "F.Cu") (net 26))
   (segment (start 15.85 52) (end 9.35 52) (width 0.25) (layer "F.Cu") (net 26))
@@
   (segment (start 51.56 2.7) (end 50.385489 3.874511) (width 0.25) (layer "B.Cu") (net 26))
   (segment (start 18.2 52) (end 15.85 52) (width 0.25) (layer "B.Cu") (net 26))
+  (segment (start 33.55048 40.685238) (end 32.235718 42) (width 0.25) (layer "F.Cu") (net 27))
   (segment (start 28.05048 22.936198) (end 33.55048 28.436198) (width 0.25) (layer "F.Cu") (net 27))
+  (segment (start 28.05048 7.13048) (end 28.05048 22.936198) (width 0.25) (layer "F.Cu") (net 27))
+  (segment (start 21.25 42) (end 18.7 44.55) (width 0.25) (layer "F.Cu") (net 27))
   (segment (start 26.16 5.24) (end 28.05048 7.13048) (width 0.25) (layer "F.Cu") (net 27))
   (segment (start 32.235718 42) (end 21.25 42) (width 0.25) (layer "F.Cu") (net 27))
-  (segment (start 33.55048 40.685238) (end 32.235718 42) (width 0.25) (layer "F.Cu") (net 27))
-  (segment (start 21.25 42) (end 18.7 44.55) (width 0.25) (layer "F.Cu") (net 27))
+  (segment (start 33.55048 28.436198) (end 33.55048 40.685238) (width 0.25) (layer "F.Cu") (net 27))
   (segment (start 18.7 44.55) (end 15.875 44.55) (width 0.25) (layer "F.Cu") (net 27))
-  (segment (start 33.55048 28.436198) (end 33.55048 40.685238) (width 0.25) (layer "F.Cu") (net 27))
   (segment (start 56.625 37.25) (end 56.525 37.15) (width 0.25) (layer "F.Cu") (net 28))
   (segment (start 62.70144 13.858594) (end 62.70144 33.04856) (width 0.25) (layer "F.Cu") (net 28))
@@
   (segment (start 62.0524 15.761215) (end 62.0524 39.904728) (width 0.25) (layer "B.Cu") (net 32))
   (segment (start 31.3 29.5) (end 29 29.5) (width 0.25) (layer "B.Cu") (net 32))
-  (segment (start 26.2 7.8) (end 23.64 7.8) (width 0.25) (layer "F.Cu") (net 33))
-  (segment (start 23.64 7.8) (end 21.08 5.24) (width 0.25) (layer "F.Cu") (net 33))
-  (segment (start 29.85048 37.2) (end 32.55048 34.5) (width 0.25) (layer "F.Cu") (net 33))
-  (segment (start 32.55048 34.5) (end 32.55048 28.707634) (width 0.25) (layer "F.Cu") (net 33))
-  (segment (start 29.025 37.2) (end 29.85048 37.2) (width 0.25) (layer "F.Cu") (net 33))
-  (segment (start 32.55048 28.707634) (end 27 23.157154) (width 0.25) (layer "F.Cu") (net 33))
-  (segment (start 27 8.6) (end 26.2 7.8) (width 0.25) (layer "F.Cu") (net 33))
+  (segment (start 27 23.157154) (end 32.55048 28.707634) (width 0.25) (layer "F.Cu") (net 33))
+  (segment (start 27 8.6) (end 27 23.157154) (width 0.25) (layer "F.Cu") (net 33))
+  (segment (start 26.2 7.8) (end 27 8.6) (width 0.25) (layer "F.Cu") (net 33))
+  (segment (start 29.85048 37.2) (end 29.025 37.2) (width 0.25) (layer "F.Cu") (net 33))
+  (segment (start 32.55048 28.707634) (end 32.55048 34.5) (width 0.25) (layer "F.Cu") (net 33))
+  (segment (start 32.55048 34.5) (end 29.85048 37.2) (width 0.25) (layer "F.Cu") (net 33))
+  (segment (start 23.64 7.8) (end 26.2 7.8) (width 0.25) (layer "F.Cu") (net 33))
+  (segment (start 21.08 5.24) (end 23.64 7.8) (width 0.25) (layer "F.Cu") (net 33))
   (segment (start 8.25 24.625) (end 8.25 28.45) (width 0.25) (layer "F.Cu") (net 34))
   (segment (start 9.35 29.55) (end 15.85 29.55) (width 0.25) (layer "F.Cu") (net 34))
@@
   (segment (start 62.50192 40.090926) (end 58.984745 43.608101) (width 0.25) (layer "B.Cu") (net 34))
   (segment (start 22.80048 41.55048) (end 18.4 37.15) (width 0.25) (layer "F.Cu") (net 35))
+  (segment (start 27.839282 23.360718) (end 29.339282 24.860718) (width 0.25) (layer "F.Cu") (net 35))
+  (segment (start 27.6 23.121436) (end 27.839282 23.360718) (width 0.25) (layer "F.Cu") (net 35))
   (segment (start 32.04952 41.55048) (end 31.64952 41.55048) (width 0.25) (layer "F.Cu") (net 35))
+  (segment (start 27.6 7.8) (end 27.6 23.121436) (width 0.25) (layer "F.Cu") (net 35))
   (segment (start 27.05 7.25) (end 27.6 7.8) (width 0.25) (layer "F.Cu") (net 35))
   (segment (start 23.62 5.24) (end 25.63 7.25) (width 0.25) (layer "F.Cu") (net 35))
@@
   (segment (start 29.339282 24.860718) (end 33.05048 28.571916) (width 0.25) (layer "F.Cu") (net 35))
   (segment (start 18.4 37.15) (end 15.875 37.15) (width 0.25) (layer "F.Cu") (net 35))
+  (segment (start 27.6 23.121435) (end 27.839282 23.360718) (width 0.25) (layer "F.Cu") (net 35))
   (segment (start 25.63 7.25) (end 27.05 7.25) (width 0.25) (layer "F.Cu") (net 35))
   (segment (start 33.05048 28.571916) (end 33.05048 40.54952) (width 0.25) (layer "F.Cu") (net 35))
-  (segment (start 27.6 23.121435) (end 29.339282 24.860718) (width 0.25) (layer "F.Cu") (net 35))
   (segment (start 8.38 2.7) (end 10.92 2.7) (width 0.25) (layer "F.Cu") (net 36))
   (zone (net 1) (net_name "GND") (layer "F.Cu") (hatch edge 0.508)

Commit message: some bugfixing
Parts:
- R11, R12, R13, R14, R15, R16, R17: value 150 -> 200
Changed lines of the file:
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@@
   (net 40 "unconnected-(J1-Pad12)")
   (net 41 "unconnected-(J1-Pad16)")
-  (net 42 "unconnected-(J1-Pad22)")
-  (net 43 "unconnected-(J1-Pad21)")
-  (net 44 "unconnected-(J1-Pad26)")
-  (net 45 "unconnected-(J1-Pad18)")
+  (net 42 "unconnected-(J1-Pad18)")
+  (net 43 "unconnected-(J1-Pad26)")
+  (net 44 "unconnected-(J1-Pad21)")
+  (net 45 "unconnected-(J1-Pad22)")
   (net 46 "unconnected-(J1-Pad40)")
   (footprint "HWP:PiHeader" locked (layer "F.Cu")
@@
       (net 2 "+3V3") (pinfunction "3.3V") (pintype "power_in"))
     (pad "18" thru_hole oval locked (at 2.54 20.32 90) (size 1.7 1.7) (drill 1) (layers *.Cu *.Mask)
-      (net 45 "unconnected-(J1-Pad18)") (pinfunction "BCM24") (pintype "bidirectional+no_connect"))
+      (net 42 "unconnected-(J1-Pad18)") (pinfunction "BCM24") (pintype "bidirectional+no_connect"))
     (pad "19" thru_hole oval locked (at 0 22.86 90) (size 1.7 1.7) (drill 1) (layers *.Cu *.Mask)
       (net 25 "Diode 6") (pinfunction "BCM10_MOSI") (pintype "bidirectional"))
@@
       (net 1 "GND") (pinfunction "GND") (pintype "power_in"))
     (pad "21" thru_hole oval locked (at 0 25.4 90) (size 1.7 1.7) (drill 1) (layers *.Cu *.Mask)
-      (net 43 "unconnected-(J1-Pad21)") (pinfunction "BCM9_MISO") (pintype "bidirectional+no_connect"))
+      (net 44 "unconnected-(J1-Pad21)") (pinfunction "BCM9_MISO") (pintype "bidirectional+no_connect"))
     (pad "22" thru_hole oval locked (at 2.54 25.4 90) (size 1.7 1.7) (drill 1) (layers *.Cu *.Mask)
-      (net 42 "unconnected-(J1-Pad22)") (pinfunction "BCM25") (pintype "bidirectional+no_connect"))
+      (net 45 "unconnected-(J1-Pad22)") (pinfunction "BCM25") (pintype "bidirectional+no_connect"))
     (pad "23" thru_hole oval locked (at 0 27.94 90) (size 1.7 1.7) (drill 1) (layers *.Cu *.Mask)
       (net 28 "Diode 4") (pinfunction "BCM11_SCLK") (pintype "bidirectional"))
@@
       (net 1 "GND") (pinfunction "GND") (pintype "power_in"))
     (pad "26" thru_hole oval locked (at 2.54 30.48 90) (size 1.7 1.7) (drill 1) (layers *.Cu *.Mask)
-      (net 44 "unconnected-(J1-Pad26)") (pinfunction "BCM7_CE1") (pintype "bidirectional+no_connect"))
+      (net 43 "unconnected-(J1-Pad26)") (pinfunction "BCM7_CE1") (pintype "bidirectional+no_connect"))
     (pad "27" thru_hole oval locked (at 0 33.02 90) (size 1.7 1.7) (drill 1) (layers *.Cu *.Mask)
       (net 24 "Diode 7") (pinfunction "BCM0_ID_SD") (pintype "bidirectional"))
@@
       (effects (font (size 1 1) (thickness 0.15)))
     )
-    (fp_text value "150" (at 0 1.65) (layer "F.Fab") hide
+    (fp_text value "200" (at 0 1.65) (layer "F.Fab") hide
       (effects (font (size 1 1) (thickness 0.15)))
     )
@@
       (effects (font (size 1 1) (thickness 0.15)))
     )
-    (fp_text value "150" (at 0 1.65) (layer "F.Fab") hide
+    (fp_text value "200" (at 0 1.65) (layer "F.Fab") hide
       (effects (font (size 1 1) (thickness 0.15)))
     )
@@
       (effects (font (size 1 1) (thickness 0.15)))
     )
-    (fp_text value "150" (at 0 1.65) (layer "F.Fab") hide
+    (fp_text value "200" (at 0 1.65) (layer "F.Fab") hide
       (effects (font (size 1 1) (thickness 0.15)))
     )
@@
       (effects (font (size 1 1) (thickness 0.15)))
     )
-    (fp_text value "150" (at 0 1.65) (layer "F.Fab") hide
+    (fp_text value "200" (at 0 1.65) (layer "F.Fab") hide
       (effects (font (size 1 1) (thickness 0.15)))
     )
@@
       (effects (font (size 1 1) (thickness 0.15)))
     )
-    (fp_text value "150" (at 0 1.65) (layer "F.Fab") hide
+    (fp_text value "200" (at 0 1.65) (layer "F.Fab") hide
       (effects (font (size 1 1) (thickness 0.15)))
     )
@@
       (effects (font (size 1 1) (thickness 0.15)))
     )
-    (fp_text value "150" (at 0 1.65) (layer "F.Fab") hide
+    (fp_text value "200" (at 0 1.65) (layer "F.Fab") hide
       (effects (font (size 1 1) (thickness 0.15)))
     )
@@
       (effects (font (size 1 1) (thickness 0.15)))
     )
-    (fp_text value "150" (at 0 1.65) (layer "F.Fab") hide
-      (effects (font (size 1 1) (thickness 0.15)))
-    )
+    (fp_text value "200" (at 0 1.65) (layer "F.Fab") hide
+      (effects (font (size 1 1) (thickness 0.15)))
+    )

Commit message: last minor changes
Parts:
- R11, R12, R13, R14, R15, R16, R17: value 200 -> 330
- R18: value 150 -> 330
Connections:
- J1 pad 21: unconnected-(J1-Pad21) -> Diode 4
- J1 pad 23: Diode 4 -> Diode 3
- J1 pad 24: Diode 3 -> Diode 7
- J1 pad 27: Diode 7 -> unconnected-(J1-Pad27)
- J1 pad 28: Diode 8 -> unconnected-(J1-Pad28)
- J1 pad 40: unconnected-(J1-Pad40) -> Diode 8
Routing:
- net Diode 8: track 64.1 -> 51.4 mm
- net Diode 7: track 75.0 -> 82.3 mm
- net SCL: track 55.6 -> 61.0 mm
- net Diode 4: track 57.1 -> 59.6 mm
- net Diode 3: track 81.6 -> 79.6 mm
- net SDA: track 66.1 -> 67.1 mm
- net GND: vias 1 -> 4
