File: board/RPi_Hat.kicad_sch (KiCad schematic)
At the start: 42 parts, among them J1 PiHat, Q1 PMOS_GSD, SW1 Pushbutton, SW2 Pushbutton, SW3 Pushbutton, SW4 Pushbutton, SW5 Pushbutton, SW6 Pushbutton, SW7 Pushbutton, SW8 Pushbutton

Commit message: final version
Connections:
- net +3V3: now also Q1.2 (S)
- net GND: now also D9.1 (K)
- net SDA: now also R20.2
Changed lines of the file:
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@@
+    )
+  )
+  (global_label "SDA" (shape input) (at 53.34 165.1 0) (fields_autoplaced)
+    (effects (font (size 1.27 1.27)) (justify left))
+    (property "Intersheet References" "${INTERSHEET_REFS}" (id 0) (at 59.2323 165.1794 0)
+      (effects (font (size 1.27 1.27)) (justify left) hide)
     )
   )
@@
     (pin "2")
   )
+  (symbol (lib_id "HWP:GND") (at 38.1 185.42 0) (unit 1)
+    (in_bom yes) (on_board yes)
+    (property "Reference" "#PWR0115" (id 0) (at 38.1 191.77 0)
+      (effects (font (size 1.27 1.27)) hide)
+    )
+    (property "Value" "GND" (id 1) (at 38.227 189.8142 0))
+    (property "Footprint" "" (id 2) (at 38.1 185.42 0)
+      (effects (font (size 1.27 1.27)) hide)
+    )
+    (property "Datasheet" "" (id 3) (at 38.1 185.42 0)
+      (effects (font (size 1.27 1.27)) hide)
+    )
+    (pin "1")
+  )
   (symbol (lib_id "HWP:GND") (at 54.61 96.52 0) (unit 1)
     (in_bom yes) (on_board yes)
@@
     (pin "2")
   )
+  (symbol (lib_id "HWP:+3V3") (at 38.1 160.02 0) (unit 1)
+    (in_bom yes) (on_board yes)
+    (property "Reference" "#PWR0116" (id 0) (at 38.1 163.83 0)
+      (effects (font (size 1.27 1.27)) hide)
+    )
+    (property "Value" "+3V3" (id 1) (at 38.481 155.6258 0))
+    (property "Footprint" "" (id 2) (at 38.1 160.02 0)
+      (effects (font (size 1.27 1.27)) hide)
+    )
+    (property "Datasheet" "" (id 3) (at 38.1 160.02 0)
+      (effects (font (size 1.27 1.27)) hide)
+    )
+    (pin "1")
+  )
   (symbol (lib_id "HWP:R") (at 67.31 39.37 0) (unit 1)
     (in_bom yes) (on_board yes) (fields_autoplaced)
@@
       (reference "#PWR0114") (unit 1) (value "GND") (footprint "")
     )
+    (path "/5dcf62bc-50b1-4bd4-8570-afa9a56dc491"
+      (reference "#PWR0115") (unit 1) (value "GND") (footprint "")
+    )
+    (path "/9104b1fe-3da9-48b2-98b4-0efb1e589f26"
+      (reference "#PWR0116") (unit 1) (value "+3V3") (footprint "")
+    )
     (path "/4ec4cd79-04cf-4d0b-abf3-606c618c406d"
       (reference "A1") (unit 1) (value "Sparkfun-CCS811") (footprint "HWP:Sparkfun-CCS881")
@@
     )
     (path "/520f8c5e-956a-412c-81ca-b87c6f31092b"
-      (reference "D9") (unit 1) (value "LED") (footprint "HWP:LED_0805")
+      (reference "D9") (unit 1) (value "green") (footprint "HWP:LED_0805")
     )
     (path "/bd09a830-946b-4465-bbb8-4e67bb31c203"
@@
     )
     (path "/1da254ed-29b1-422b-95d9-60841f7f8478"
-      (reference "R19") (unit 1) (value "300") (footprint "HWP:R_0805")
+      (reference "R19") (unit 1) (value "200") (footprint "HWP:R_0805")
     )
     (path "/fd42a2ba-8b95-481f-80e3-5094be8c620b"
-      (reference "R20") (unit 1) (value "R") (footprint "HWP:R_0805")
+      (reference "R20") (unit 1) (value "100") (footprint "HWP:R_0805")
     )
     (path "/64fe4ef0-94d6-4168-93a5-da4cb1d6b68d"
